File: pcb/mp2-xc7k-test/fpgasupport.kicad_sch (KiCad schematic)
At the start: 17 parts, among them J6 XILINX_JTAG, U4 XC7K160T-1FFG676C

Commit message: Continued layout, 454 unrouted
Parts:
- U4: footprint (none) -> azonenberg_pcb:BGA_676_27x27_FULLARRAY_1MM_FFG676
Changed lines of the file:
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@@
 			)
 		)
-		(property "Footprint" ""
+		(property "Footprint" "azonenberg_pcb:BGA_676_27x27_FULLARRAY_1MM_FFG676"
 			(at 53.34 83.82 0)
 			(effects
@@
 			)
 		)
-		(property "Footprint" ""
+		(property "Footprint" "azonenberg_pcb:BGA_676_27x27_FULLARRAY_1MM_FFG676"
 			(at 187.96 167.64 0)
 			(effects
@@
 			)
 		)
-		(property "Footprint" ""
+		(property "Footprint" "azonenberg_pcb:BGA_676_27x27_FULLARRAY_1MM_FFG676"
 			(at 109.22 177.8 0)
 			(effects
