File: pcb/mp2-xc7k-test/fpga.kicad_sch (KiCad schematic)
At the start: 60 parts, among them J4 CONN_SFP_HOST, J7 SFP_CAGE, U10 SIT9121AI-2BF-XXS156.250000G, U11 ECS-1612MV-250-CN, U32 S25FL128SAGBHIA10, U4 XC7K160T-1FFG676C

Commit message: Continued layout, 454 unrouted
Parts:
- added J13: PMOD_HOST, azonenberg_pcb:CONN_HEADER_2.54MM_2x6_RA_PMOD_HOST, symbol special-azonenberg:PMOD_HOST
- added M1: 960-27-12-F-AB-0, azonenberg_pcb:HEATSINK_WAKEFIELDVETTE_960-27-12-D-AB-0, symbol special-azonenberg:MECHANICAL
- D31, D32, D33, D34, D39, D40: footprint azonenberg_pcb:EIA_0603_LED -> azonenberg_pcb:EIA_0402_LED
- U4: footprint (none) -> azonenberg_pcb:BGA_676_27x27_FULLARRAY_1MM_FFG676
Connections:
- net 3V3: now also J13.12 (3V3), J13.6 (3V3)
- net GND: now also J13.11 (GND), J13.5 (GND)
- net PCIE_REF_AC_N: now also U4.K6 (MGTREFCLK1P_115); no longer U4.K5 (MGTREFCLK1N_115)
- net PCIE_REF_AC_P: now also U4.K5 (MGTREFCLK1N_115); no longer U4.K6 (MGTREFCLK1P_115)
- net PCIE_RX_AC_N: now also U4.P1 (MGTXTXN0_115); no longer U4.M1 (MGTXTXN1_115)
- net PCIE_RX_AC_P: now also U4.P2 (MGTXTXP0_115); no longer U4.M2 (MGTXTXP1_115)
- net PCIE_TX_AC_N: now also U4.R3 (MGTXRXN0_115); no longer U4.N3 (MGTXRXN1_115)
- net PCIE_TX_AC_P: now also U4.R4 (MGTXRXP0_115); no longer U4.N4 (MGTXRXP1_115)
- net SFP_LED2: now also U4.D25 (IO_L15N_T2_DQS_DOUT_CSO_B_14); no longer U4.J25 (IO_L22N_T3_A04_D20_14)
- net SFP_RX_N: now also U4.N3 (MGTXRXN1_115); no longer U4.R3 (MGTXRXN0_115)
- net SFP_RX_P: now also U4.N4 (MGTXRXP1_115); no longer U4.R4 (MGTXRXP0_115)
- net SFP_TX_N: now also U4.M2 (MGTXTXP1_115); no longer U4.P1 (MGTXTXN0_115)
- net SFP_TX_P: now also U4.M1 (MGTXTXN1_115); no longer U4.P2 (MGTXTXP0_115)
- net FPGA_PMOD_DQ4: now reaches U4.E25 (IO_L15P_T2_DQS_RDWR_B_14)
- net FPGA_PMOD_DQ4: now also J13.7 (D4)
- net FPGA_PMOD_DQ0: now reaches U4.E26 (IO_L17N_T2_A13_D29_14)
- net FPGA_PMOD_DQ0: now also J13.1 (D0)
- net FPGA_PMOD_DQ5: now reaches U4.G25 (IO_L16P_T2_CSI_B_14)
- net FPGA_PMOD_DQ5: now also J13.8 (D5)
- net FPGA_PMOD_DQ1: now reaches U4.G26 (IO_L16N_T2_A15_D31_14)
- net FPGA_PMOD_DQ1: now also J13.2 (D1)
- net FPGA_PMOD_DQ6: now reaches U4.H26 (IO_L18N_T2_A11_D27_14)
- net FPGA_PMOD_DQ6: now also J13.9 (D6)
- net FPGA_PMOD_DQ2: now reaches U4.J24 (IO_L22P_T3_A05_D21_14)
- net FPGA_PMOD_DQ2: now also J13.3 (D2)
- net FPGA_PMOD_DQ7: now reaches U4.J26 (IO_L18P_T2_A12_D28_14)
- net FPGA_PMOD_DQ7: now also J13.10 (D7)
- new net FPGA_PMOD_DQ3: J13.4 (D3), U4.J25 (IO_L22N_T3_A04_D20_14)
- no-connect marks 65 -> 57
Other:
- note added: "Debug PMOD"
- note added: "Heatsink"
- note added: "Polarity invert"

Commit message: Continued PCB routing, 344 nets left
Connections:
- net GTX1_REF_AC_N: now also U10.4 (OUT_P); no longer U10.5 (OUT_N)
- net GTX1_REF_AC_P: now also U10.5 (OUT_N); no longer U10.4 (OUT_P)
Other:
- moved on the sheet: C76, C77
Changed lines of the file:
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@@
 	)
 	(label "GTX_REF1_N"
-		(at 92.71 36.83 0)
+		(at 92.71 26.67 0)
 		(effects
 			(font
@@
 	)
 	(label "GTX1_REF_AC_P"
-		(at 71.12 26.67 0)
+		(at 71.12 36.83 0)
 		(effects
 			(font
@@
 	)
 	(label "GTX1_REF_AC_N"
-		(at 71.12 36.83 0)
+		(at 71.12 26.67 0)
 		(effects
 			(font
@@
 	)
 	(label "GTX_REF1_P"
-		(at 92.71 26.67 0)
+		(at 92.71 36.83 0)
 		(effects
 			(font
@@
 	(symbol
 		(lib_id "device:C")
-		(at 88.9 36.83 90)
+		(at 88.9 26.67 90)
 		(unit 1)
 		(exclude_from_sim no)
@@
 		(fields_autoplaced yes)
 		(property "Reference" "C77"
-			(at 88.9 30.5265 90)
+			(at 88.9 20.3665 90)
 			(effects
 				(font
@@
 		)
 		(property "Value" "0.1 uF"
-			(at 88.9 32.9508 90)
+			(at 88.9 22.7908 90)
 			(effects
 				(font
@@
 		)
 		(property "Footprint" "azonenberg_pcb:EIA_0402_CAP_NOSILK"
-			(at 92.71 35.8648 0)
+			(at 92.71 25.7048 0)
 			(effects
 				(font
@@
 		)
 		(property "Datasheet" ""
-			(at 88.9 36.83 0)
+			(at 88.9 26.67 0)
 			(effects
 				(font
@@
 		)
 		(property "Description" "Unpolarized capacitor"
-			(at 88.9 36.83 0)
+			(at 88.9 26.67 0)
 			(effects
 				(font
@@
 	(symbol
 		(lib_id "device:C")
-		(at 88.9 26.67 90)
+		(at 88.9 36.83 90)
 		(unit 1)
 		(exclude_from_sim no)
@@
 		(fields_autoplaced yes)
 		(property "Reference" "C76"
-			(at 88.9 20.3665 90)
+			(at 88.9 30.5265 90)
 			(effects
 				(font
@@
 		)
 		(property "Value" "0.1 uF"
-			(at 88.9 22.7908 90)
+			(at 88.9 32.9508 90)
 			(effects
 				(font
@@
 		)
 		(property "Footprint" "azonenberg_pcb:EIA_0402_CAP_NOSILK"
-			(at 92.71 25.7048 0)
+			(at 92.71 35.8648 0)
 			(effects
 				(font
@@
 		)
 		(property "Datasheet" ""
-			(at 88.9 26.67 0)
+			(at 88.9 36.83 0)
 			(effects
 				(font
@@
 		)
 		(property "Description" "Unpolarized capacitor"
-			(at 88.9 26.67 0)
+			(at 88.9 36.83 0)
 			(effects
 				(font

Commit message: 111 unrouted, getting close
Connections:
- net FPGA_LED0: now also U4.J23 (IO_L24N_T3_A00_D16_14); no longer U4.L23 (IO_25_14)
- net FPGA_LED1: now also U4.K23 (IO_L24P_T3_A01_D17_14); no longer U4.J23 (IO_L24N_T3_A00_D16_14)
- net FPGA_LED2: now also U4.K22 (IO_L23N_T3_A02_D18_14); no longer U4.K23 (IO_L24P_T3_A01_D17_14)
- net FPGA_LED3: now also U4.L23 (IO_25_14); no longer U4.K22 (IO_L23N_T3_A02_D18_14)
- net SFP_LED2: now also U4.J21 (IO_L21P_T3_DQS_14); no longer U4.D25 (IO_L15N_T2_DQS_DOUT_CSO_B_14)
Changed lines of the file:
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@@
-	)
-	(no_connect
-		(at 345.44 219.71)
 	)
 	(no_connect
@@
 	(no_connect
 		(at 345.44 161.29)
+	)
+	(no_connect
+		(at 345.44 191.77)
 	)
 	(no_connect
@@
 	)
 	(label "FPGA_LED3"
-		(at 345.44 232.41 180)
+		(at 345.44 240.03 180)
 		(effects
 			(font
@@
 	)
 	(label "FPGA_LED0"
-		(at 345.44 240.03 180)
+		(at 345.44 237.49 180)
 		(effects
 			(font
@@
 	)
 	(label "SFP_LED2"
-		(at 345.44 191.77 180)
+		(at 345.44 219.71 180)
 		(effects
 			(font
@@
 	)
 	(label "FPGA_LED1"
-		(at 345.44 237.49 180)
+		(at 345.44 234.95 180)
 		(effects
 			(font
@@
 	)
 	(label "FPGA_LED2"
-		(at 345.44 234.95 180)
-		(effects
-			(font
+		(at 345.44 232.41 180)
+		(effects
+			(font

Commit message: Final MP2 XC7K test board ready for fab
Parts:
- added C142, C143: 0.47 uF, azonenberg_pcb:EIA_0402_CAP_NOSILK, symbol device:C
Connections:
- net 3V3: now also C142.1, C143.1
- net GND: now also C142.2, C143.2
Other:
- note added: "Return current for CCLK"
Changed lines of the file:
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@@
 		)
 	)
+	(text "Return current for CCLK"
+		(exclude_from_sim no)
+		(at 276.86 250.19 0)
+		(effects
+			(font
+				(size 1.27 1.27)
+			)
+		)
+	)
 	(text "Heatsink"
 		(exclude_from_sim no)
@@
 	)
 	(junction
+		(at 267.97 248.92)
+		(diameter 0)
+		(color 0 0 0 0)
+	)
+	(junction
 		(at 148.59 162.56)
 		(diameter 0)
@@
 	)
 	(junction
+		(at 248.92 241.3)
+		(diameter 0)
+		(color 0 0 0 0)
+	)
+	(junction
 		(at 217.17 187.96)
 		(diameter 0)
@@
 	)
 	(junction
+		(at 248.92 248.92)
+		(diameter 0)
+		(color 0 0 0 0)
+	)
+	(junction
+		(at 267.97 241.3)
+		(diameter 0)
+		(color 0 0 0 0)
+	)
+	(junction
 		(at 154.94 262.89)
 		(diameter 0)
@@
 	(wire
 		(pts
+			(xy 248.92 241.3) (xy 267.97 241.3)
+		)
+		(stroke
+			(width 0)
+			(type default)
+		)
+	)
+	(wire
+		(pts
 			(xy 40.64 27.94) (xy 40.64 30.48)
 		)
@@
 	(wire
 		(pts
+			(xy 267.97 241.3) (xy 283.21 241.3)
+		)
+		(stroke
+			(width 0)
+			(type default)
+		)
+	)
+	(wire
+		(pts
 			(xy 212.09 179.07) (xy 217.17 179.07)
 		)
@@
 	(wire
 		(pts
+			(xy 267.97 248.92) (xy 283.21 248.92)
+		)
+		(stroke
+			(width 0)
+			(type default)
+		)
+	)
+	(wire
+		(pts
 			(xy 121.92 187.96) (xy 148.59 187.96)
 		)
@@
 		)
 	)
+	(wire
+		(pts
+			(xy 248.92 248.92) (xy 267.97 248.92)
+		)
+		(stroke
+			(width 0)
+			(type default)
+		)
+	)
 	(polyline
 		(pts
@@
 	)
 	(symbol
+		(lib_id "device:C")
+		(at 283.21 245.11 0)
+		(unit 1)
+		(exclude_from_sim no)
+		(in_bom yes)
+		(on_board yes)
+		(dnp no)
+		(property "Reference" "C143"
+			(at 286.131 243.9416 0)
+			(effects
+				(font
+					(size 1.27 1.27)
+				)
+				(justify left)
+			)
+		)
+		(property "Value" "0.47 uF"
+			(at 286.131 246.253 0)
+			(effects
+				(font
+					(size 1.27 1.27)
+				)
+				(justify left)
+			)
+		)
+		(property "Footprint" "azonenberg_pcb:EIA_0402_CAP_NOSILK"
+			(at 284.1752 248.92 0)
+			(effects
+				(font
+					(size 1.27 1.27)
+				)
+				(hide yes)
+			)
+		)
+		(property "Datasheet" ""
+			(at 283.21 245.11 0)
+			(effects
+				(font
+					(size 1.27 1.27)
+				)
+				(hide yes)
+			)
+		)
+		(property "Description" ""
+			(at 283.21 245.11 0)
+			(effects
+				(font
+					(size 1.27 1.27)
+				)
+				(hide yes)
+			)
+		)
+		(pin "1"
+		)
+		(pin "2"
+		)
+		(instances
+			(project "mp2-xc7k-test"
+				(path "/b52ad5ff-5dbb-4f64-8839-2dc6cd4521cb/4d79ff40-6c61-41c3-bba8-95e178d9ca85"
+					(reference "C143")
+					(unit 1)
+				)
+			)
+		)
+	)
+	(symbol
 		(lib_id "xilinx-azonenberg:XC7KxT-FFG676")
 		(at 350.52 241.3 0)
@@
 					(unit 1)
 				)
+			)
+		)
+	)
+	(symbol
+		(lib_id "device:C")
+		(at 267.97 245.11 0)
+		(unit 1)
+		(exclude_from_sim no)
+		(in_bom yes)
+		(on_board yes)
+		(dnp no)
+		(property "Reference" "C142"
+			(at 270.891 243.9416 0)
+			(effects
+				(font
+					(size 1.27 1.27)
+				)
+				(justify left)
+			)
+		)
+		(property "Value" "0.47 uF"
+			(at 270.891 246.253 0)
+			(effects
+				(font
+					(size 1.27 1.27)
+				)
+				(justify left)
+			)
+		)
+		(property "Footprint" "azonenberg_pcb:EIA_0402_CAP_NOSILK"
+			(at 268.9352 248.92 0)
+			(effects
+				(font
+					(size 1.27 1.27)
+				)
+				(hide yes)
+			)
+		)
+		(property "Datasheet" ""
+			(at 267.97 245.11 0)
+			(effects
+				(font
+					(size 1.27 1.27)
+				)
+				(hide yes)
+			)
+		)
+		(property "Description" ""
+			(at 267.97 245.11 0)
+			(effects
+				(font
+					(size 1.27 1.27)
+				)
+				(hide yes)
+			)
+		)
+		(pin "1"
+		)
+		(pin "2"
+		)
+		(instances
+			(project "mp2-xc7k-test"
+				(path "/b52ad5ff-5dbb-4f64-8839-2dc6cd4521cb/4d79ff40-6c61-41c3-bba8-95e178d9ca85"
+					(reference "C142")
+					(unit 1)
+				)

Commit message: Fixed bad pullup value. Added PnP fixture
Parts:
- R38: value 10K -> 1K
Changed lines of the file:
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@@
 			)
 		)
-		(property "Value" "10K"
+		(property "Value" "1K"
 			(at 337.82 128.27 90)
 			(effects
